File: A1.kicad_sch (KiCad schematic)
At the start: 0 parts

Commit message: A1/sch: adjust title block
Other:
- note added: "Генератор на еталонна честота, Делител, Комутатор"
- title: (none) -> Синтезатор на честота, Радио/1990/1,2,3
Changed lines of the file:
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@@
 (kicad_sch (version 20211123) (generator eeschema)
   (paper "A4")
+  (title_block
+    (title "Синтезатор на честота, Радио/1990/1,2,3")
+  )
+  (text "Генератор на еталонна честота, Делител, Комутатор" (at 178.435 175.26 0)
+    (effects (font (size 2.56 2.56)) (justify left bottom))
+  )
 )

Commit message: Update to kicad7; flush WIP
Parts:
- added C3: 200, symbol Device:C_Small
- added C5: 33uF 6V, symbol Device:C_Polarized
- added C51: 300uF 15V, symbol Device:C_Polarized
- added C52: 150nF, symbol Device:C_Small
- added DD1: К155ЛА3, symbol ГОСТ 2.743:4xNAND
- added L4: 250uH, symbol Device:L_Ferrite
- added R10001: 0, symbol Device:R_Small
- added R25: 4.7K, symbol Device:R_Potentiometer
Connections:
- new net: C51.1, C52.1, DD1.14 (VCC), L4.2
- new net: C5.2, DD1.1, DD1.2, R25.1
- new net: C3.1, DD1.8, R25.2, R25.3
- new net: DD1.3, DD1.4, DD1.5
- new net: C3.2, DD1.12, DD1.13
- new net: C5.1, DD1.10, DD1.6, DD1.9
- new net +5V: L4.1
- new net GND: R10001.1
- new net GNDD: C51.2, C52.2, DD1.7 (GND), R10001.2
- no-connect marks 0 -> 1

Commit message: Flush WIP
Parts:
- added C3 (x2), C52: 150nF, symbol Device:C_Small
- added C51: 300uF 15V, symbol Device:C_Polarized
- added DD2, DD3: К155ЛА3, symbol ladihw:К155ЛА3
- added DD4, DD5, DD6: К155ТМ2, symbol ladihw:К155ТМ2
- added DD7: К155ИЕ7, symbol ladihw:К155ИЕ7
- added R23, R24: 1K, symbol GOST-2.728:R_0125W_GOST
- added R26: 200, symbol GOST-2.728:R_0125W_GOST
- added R27: 240, symbol GOST-2.728:R_0125W_GOST
- R25: symbol Device:R_Potentiometer -> GOST-2.728:R_Potentiometer_GOST
Connections:
- net GNDD: now also C3.1, C3.1, C52.2, DD2.7 (GND), DD7.1 (D2), DD7.10 (D4), DD7.15 (D1), DD7.9 (D8), R26.1, R27.1
- net at C51.1, C52.1, DD1.14 (VCC)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: now also C52.1, DD2.14 (VCC)
- net at DD1.11: now also DD3.12, DD3.13
- net at C3.2, DD1.12, DD1.13: now also R26.2
- new net: C51.2, DD7.14 (R), R27.2
- new net: DD3.3, DD7.4 (-1)
- new net: DD3.6, DD7.5 (+1)
- new net: DD2.12, DD2.13, DD2.8
- new net: DD2.3, DD3.2
- new net: DD3.1, DD3.11, DD3.4
- new net: DD2.6, DD3.5
- new net 1: C51.1, R23.1, R24.1
- new net 17: C3.2, DD2.4, DD2.5, R24.2
- new net 18: C3.2, DD2.1, DD2.2, R23.2
- new net 19: DD7.3 (Q1)
- new net 20: DD7.2 (Q2)
- new net 21: DD7.6 (Q4)
- new net 22: DD7.7 (Q8)
- no-connect marks 1 -> 3
Other:
- moved on the sheet: C3, C5, C51, C52, DD1A, DD1B, DD1C, DD1D, DD1E, L4
